File: pcb/rev1/volume-mixer.kicad_pcb (KiCad board)
At the start: 4 copper layers, 120 x 150 mm, 162 parts, among them CON1 TC2030-IDC, J1 Conn_01x04_Pin, J10 Conn_01x04_Pin, J2 Conn_01x10_Pin, J3 Conn_01x10_Pin, J4 Conn_01x04_Pin, J5 JST, J6 Conn_01x04_Pin, J7 Conn_01x04_Pin, J8 Conn_01x04_Pin, J9 Conn_01x04_Pin, Q1 NMOS, Q10 NMOS, Q3 NMOS, Q7 NMOS, Q8 NMOS, Q9 NMOS, SW1 SW_Push, SW2 SW_Push, SW3 SW_Push, U1 STM32F302C8Tx, U2 24LC64, U3 XC6206PxxxMR, U4 XC6206PxxxMR, U5 PRTR5V0U2X, U6 TCA9548APWR, U7 TL084, U8 TL084, Y1 8MHz

Commit message: BIDIBOU
Parts:
- removed D2, D6, D7, D9: LED, A_Please:LED C516299
- D1, D10, D11, D12, D13: moved to F.Cu
- moved U2 279.6 mm to (100.1, 157.5), turned to 0 degrees
- moved C12 271.4 mm to (108.6, 159.4)
- moved C20 261.0 mm to (108.4, 127.7), turned to 0 degrees
- moved U4 258.2 mm to (108.5, 124.4), turned to 90 degrees
- moved U3 256.4 mm to (99.4, 124.5), turned to 90 degrees
- moved C17 256.2 mm to (102.0, 124.1), turned to -90 degrees
- moved C19 254.2 mm to (111.2, 124.1), turned to -90 degrees
- moved C18 254.1 mm to (99.4, 127.6), turned to 0 degrees
- moved C8 241.7 mm to (102.2, 132.2)
- moved Y1 237.6 mm to (102.1, 134.4), turned to 0 degrees
- moved R15 184.0 mm to (69.1, 149.7)
- moved R61 178.5 mm to (68.9, 158.1)
- moved R62 178.1 mm to (68.9, 159.6), turned to 0 degrees
- moved D10 177.9 mm to (82.0, 171.0)
- moved R63 173.5 mm to (72.7, 159.6), turned to 0 degrees
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Connections:
- C32 pad 1: Net-(U7A-+) -> Net-(U8A-+)
- C42 pad 1: Net-(U7C-+) -> Net-(U7A-+)
- R41 pad 2: Net-(U7A-+) -> Net-(U8A-+)
- R46 pad 2: Net-(U8A-+) -> Net-(U7B-+)
- R47 pad 1: Net-(U8A-+) -> Net-(U7B-+)
- R49 pad 2: Net-(U7B-+) -> Net-(U7C-+)
- R51 pad 1: Net-(U7B-+) -> Net-(U7C-+)
- R59 pad 2: Net-(U7C-+) -> Net-(U7A-+)
- U1 pad 19: Mute3Led -> Mute4Led
- U1 pad 20: Mute4Led -> Mute3Led
- U7 pad 1: Slider0 -> Slider4
- U7 pad 2: Slider0 -> Slider4
- U7 pad 6: Vref digi -> Vref USB
- U7 pad 7: Vref digi -> Vref USB
- U7 pad 8: Slider4 -> Vref digi
- U7 pad 9: Slider4 -> Vref digi
- U8 pad 1: Vref USB -> Slider0
- U8 pad 2: Vref USB -> Slider0
Routing:
- net D-: track 0.00 -> 155.4 mm, vias 0 -> 2
- net D+: track 0.00 -> 154.7 mm, vias 0 -> 2
- net VBUS: track 0.00 -> 128.6 mm
- net Mute4Led: track 0.00 -> 64.4 mm, vias 0 -> 2
- net Mute2Led: track 0.00 -> 50.3 mm, vias 0 -> 2
- net Net-(D11-A): track 0.00 -> 49.8 mm, vias 0 -> 1
- net Mute3Led: track 0.00 -> 49.7 mm, vias 0 -> 2
- net Mute1Led: track 0.00 -> 49.4 mm, vias 0 -> 4
- net Net-(D11-K): track 0.00 -> 43.1 mm, vias 0 -> 1
- net Mute0Led: track 2.83 -> 45.9 mm, vias 0 -> 4
- net Net-(D12-A): track 0.00 -> 31.1 mm, vias 0 -> 1
- net Net-(D13-A): track 0.00 -> 26.5 mm, vias 0 -> 1
- net Net-(D10-A): track 0.00 -> 26.1 mm, vias 0 -> 1
- net Net-(D3-A): track 0.00 -> 26.0 mm, vias 0 -> 1
- net Net-(D12-K): track 0.00 -> 25.9 mm, vias 0 -> 1
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
Commit message: BIDIBOU
Parts:
- moved U6 164.5 mm to (104.1, 73.0), turned to -90 degrees
- moved R51 121.6 mm to (145.9, 114.7)
- moved R49 121.6 mm to (145.9, 113.1), turned to 0 degrees
- moved R54 120.5 mm to (150.2, 113.1), turned to 0 degrees
- moved R53 119.2 mm to (150.2, 114.7)
- moved R47 117.7 mm to (145.9, 128.4)
- moved R46 117.6 mm to (145.9, 126.9), turned to 0 degrees
- moved U7 108.0 mm to (148.0, 120.9), turned to 90 degrees
- moved C34 105.2 mm to (148.0, 130.8), turned to -90 degrees
- moved C33 104.4 mm to (126.0, 109.7), turned to 90 degrees
- moved U8 102.4 mm to (126.0, 120.9), turned to -90 degrees
- moved R41 64.9 mm to (123.9, 113.5), turned to 0 degrees
- moved C32 64.4 mm to (123.9, 112.0)
- moved R16 61.5 mm to (220.0, 98.6)
- moved R19 61.5 mm to (220.0, 101.5)
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Routing:
- net Vana: track 14.4 -> 191.2 mm, vias 0 -> 10
- net VBUS: track 128.6 -> 256.6 mm, vias 0 -> 9
- net Net-(R41-Pad1): track 0.00 -> 85.7 mm, vias 0 -> 3
- net Net-(R50-Pad1): track 0.00 -> 73.9 mm, vias 0 -> 1
- net Net-(R44-Pad1): track 0.00 -> 73.1 mm, vias 0 -> 6
- net /SD4: track 0.00 -> 60.2 mm, vias 0 -> 1
- net /SC4: track 0.00 -> 58.3 mm, vias 0 -> 1
- net Vref ana: track 3.12 -> 59.0 mm, vias 1 -> 4
- net Slider4: track 1.59 -> 56.4 mm, vias 1 -> 4
- net /SC0: track 0.00 -> 53.5 mm
- net /SD0: track 0.00 -> 52.2 mm, vias 0 -> 1
- net Vref digi: track 2.92 -> 54.9 mm, vias 1 -> 4
- net Net-(R59-Pad1): track 0.00 -> 48.7 mm, vias 0 -> 1
- net Net-(R56-Pad1): track 0.00 -> 48.1 mm, vias 0 -> 2
- net Vref USB: track 2.65 -> 48.7 mm, vias 1 -> 4
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
Commit message: BIDIBOU
Parts:
- added C43: 100nF, Capacitor_SMD:C_0603_1608Metric, F.Cu at (215.3, 67.8)
- added C44: 100nF, Capacitor_SMD:C_0603_1608Metric, F.Cu at (223.2, 50.7)
- added C45: 100nF, Capacitor_SMD:C_0603_1608Metric, F.Cu at (223.2, 53.2)
- added C46: 100nF, Capacitor_SMD:C_0603_1608Metric, F.Cu at (223.2, 55.7)
- added C47: 100nF, Capacitor_SMD:C_0603_1608Metric, F.Cu at (223.2, 58.2)
- added C48: 100nF, Capacitor_SMD:C_0603_1608Metric, F.Cu at (223.2, 60.8)
- added C49: 100nF, Capacitor_SMD:C_0603_1608Metric, F.Cu at (223.2, 63.3)
- added C50: 100nF, Capacitor_SMD:C_0603_1608Metric, F.Cu at (223.2, 65.8)
- added C51: 100nF, Capacitor_SMD:C_0603_1608Metric, F.Cu at (231.8, 52.1)
- added C52: 100nF, Capacitor_SMD:C_0603_1608Metric, F.Cu at (231.8, 54.6)
- added C53: 100nF, Capacitor_SMD:C_0603_1608Metric, F.Cu at (231.8, 57.1)
- added C54: 100nF, Capacitor_SMD:C_0603_1608Metric, F.Cu at (231.8, 59.6)
- added C55: 100nF, Capacitor_SMD:C_0603_1608Metric, F.Cu at (231.8, 62.1)
- added C56: 100nF, Capacitor_SMD:C_0603_1608Metric, F.Cu at (231.8, 64.6)
- R11, R12, U5, USB1: moved to F.Cu
- moved C21 136.8 mm to (58.0, 48.1)
- moved C22 136.8 mm to (58.0, 49.6)
- moved R25 126.8 mm to (61.8, 48.9), turned to 90 degrees
- moved R24 124.8 mm to (63.3, 48.9), turned to 90 degrees
- moved C23 114.6 mm to (79.9, 48.1)
- moved C24 114.6 mm to (79.9, 49.6)
- moved R39 111.1 mm to (111.2, 69.5), turned to -90 degrees
- moved R27 110.5 mm to (83.9, 48.9), turned to 90 degrees
- moved R38 109.5 mm to (112.7, 69.5), turned to -90 degrees
- moved R26 108.5 mm to (85.4, 48.9), turned to 90 degrees
- moved R37 103.6 mm to (114.2, 69.5), turned to -90 degrees
- moved R17 103.3 mm to (100.6, 79.0), turned to 90 degrees
- moved R36 102.0 mm to (115.8, 69.5), turned to -90 degrees
- moved R18 101.3 mm to (102.2, 79.0), turned to 90 degrees
- moved CON1 98.3 mm to (49.6, 121.6), turned to 90 degrees
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Connections:
- J1 pad 1: +3V3 -> VBUS
- J1 pad 3: VBUS -> +3V3
- U5 pad 2: D- -> D+
- U5 pad 3: D+ -> D-
Routing:
- net /SDA: track 13.0 -> 126.3 mm, vias 2 -> 3
- net /SCL: track 16.5 -> 127.8 mm
- net +3V3: track 8.10 -> 74.0 mm
- net D-: track 146.8 -> 130.0 mm, vias 4 -> 2
- net /SD5: track 0.00 -> 16.0 mm
- net /SC5: track 0.00 -> 15.1 mm
- net D+: track 145.8 -> 131.3 mm, vias 4 -> 2
- net /SD6: track 0.00 -> 14.0 mm
- net /RESET: track 3.02 -> 16.2 mm
- net /SC6: track 0.00 -> 12.7 mm
- net /SD7: track 0.00 -> 11.9 mm
- net /SC7: track 0.00 -> 11.1 mm
- net /SWCLK: track 2.82 -> 12.7 mm
- net /SC3: track 34.8 -> 43.7 mm
- net /SWDIO: track 2.24 -> 8.80 mm
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- removed copper zone on In2.Cu, net GND

Commit message: BIDIBOU
Parts:
- removed the C13 at (195.0, 122.3)
- removed the C14 at (217.8, 120.0)
- removed the C43 at (215.3, 67.8)
- removed the C44 at (223.2, 50.7)
- removed the C45 at (223.2, 53.2)
- removed the C47 at (223.2, 58.2)
- removed the C48 at (223.2, 60.8)
- removed the C49 at (223.2, 63.3)
- removed the C50 at (223.2, 65.8)
- removed the C51 at (231.8, 52.1)
- removed the C52 at (231.8, 54.6)
- removed the C53 at (231.8, 57.1)
- removed the C54 at (231.8, 59.6)
- removed the C55 at (231.8, 62.1)
- removed the C56 at (231.8, 64.6)
- removed the C9 at (182.8, 121.2)
- removed the Q1 at (209.1, 120.1)
- removed the R1 at (186.9, 121.2)
- removed the R13 at (208.7, 102.3)
- removed the R16 at (220.0, 98.6)
- removed the R19 at (220.0, 101.5)
- removed the R2 at (198.6, 122.3)
- removed the R3 at (218.5, 126.2)
- removed the R4 at (218.6, 128.3)
- removed the R5 at (213.6, 120.1)
- added C1: 100nF, Capacitor_SMD:C_0603_1608Metric, B.Cu at (107.0, 39.4)
- added C15: 100nF, Capacitor_SMD:C_0603_1608Metric, B.Cu at (53.4, 121.9)
- added C17: 100nF, Capacitor_SMD:C_0603_1608Metric, B.Cu at (157.2, 98.0)
- added C19: 100nF, Capacitor_SMD:C_0603_1608Metric, B.Cu at (158.0, 94.2)
- added C2: 100nF, Capacitor_SMD:C_0603_1608Metric, B.Cu at (105.5, 39.4)
- added C22: 100nF, Capacitor_SMD:C_0603_1608Metric, B.Cu at (80.8, 129.9)
- added C23: 4,7uF, Capacitor_SMD:C_0603_1608Metric, B.Cu at (91.8, 50.7)
- added C25: 470nF, Capacitor_SMD:C_0603_1608Metric, B.Cu at (87.3, 55.0)
- added C26: 100nF, Capacitor_SMD:C_0603_1608Metric, B.Cu at (53.4, 129.3)
- added C27: 100nF, Capacitor_SMD:C_0603_1608Metric, B.Cu at (157.2, 104.2)
- added C3: 100nF, Capacitor_SMD:C_0603_1608Metric, B.Cu at (68.3, 147.1)
- added C32: 100nF, Capacitor_SMD:C_0603_1608Metric, F.Cu at (76.4, 42.0)
- added C33: 100nF, Capacitor_SMD:C_0603_1608Metric, F.Cu at (65.6, 42.0)
- added C34: 100nF, Capacitor_SMD:C_0603_1608Metric, F.Cu at (67.0, 46.3)
- added C4: 100nF, Capacitor_SMD:C_0603_1608Metric, B.Cu at (71.8, 147.1)
- added C5: 100nF, Capacitor_SMD:C_0603_1608Metric, B.Cu at (135.3, 145.5)
- added C6: 100nF, Capacitor_SMD:C_0603_1608Metric, B.Cu at (138.9, 145.5)
- added C7: 100nF, Capacitor_SMD:C_0603_1608Metric, B.Cu at (157.9, 151.2)
- added D2: LED, LED_SMD:LED_0805_2012Metric, B.Cu at (161.1, 117.0)
- added Q6: NMOS, Package_TO_SOT_SMD:SOT-23, B.Cu at (111.6, 56.4)
- added Q7: NMOS, Package_TO_SOT_SMD:SOT-23, B.Cu at (115.0, 56.4)
- added Q8: NMOS, Package_TO_SOT_SMD:SOT-23, B.Cu at (118.4, 56.4)
- added Q9: NMOS, Package_TO_SOT_SMD:SOT-23, B.Cu at (90.7, 55.0)
- added R20: 100, Resistor_SMD:R_0603_1608Metric, B.Cu at (110.7, 60.9)
- added R21: 100, Resistor_SMD:R_0603_1608Metric, B.Cu at (114.1, 60.9)
- added R23: 10K, Resistor_SMD:R_0603_1608Metric, B.Cu at (112.2, 60.9)
- added R24: 10K, Resistor_SMD:R_0603_1608Metric, B.Cu at (115.6, 60.9)
- added R25: 10K, Resistor_SMD:R_0603_1608Metric, B.Cu at (119.1, 60.9)
- added R26: 10k, Resistor_SMD:R_0603_1608Metric, B.Cu at (83.8, 129.1)
- added R27: 10K, Resistor_SMD:R_0603_1608Metric, B.Cu at (85.8, 55.0)
- added R28: 10K, Resistor_SMD:R_0603_1608Metric, B.Cu at (93.3, 50.7)
- added R29: 100k, Resistor_SMD:R_0603_1608Metric, B.Cu at (93.5, 55.1)
- added R37: 10k, Resistor_SMD:R_0603_1608Metric, B.Cu at (133.9, 51.9)
- added R6: 1k2, Resistor_SMD:R_0603_1608Metric, B.Cu at (161.1, 118.9)
- added R7: 150, Resistor_SMD:R_0603_1608Metric, B.Cu at (113.5, 45.3)
- added R8: 95, Resistor_SMD:R_0603_1608Metric, B.Cu at (115.0, 45.3)
- added R9: 95, Resistor_SMD:R_0603_1608Metric, B.Cu at (116.5, 45.3)
- C16: value 470nF -> 100nF
- C46: moved to B.Cu
- D1: value LED -> LED_ARGB; footprint A_Please:LED C516299 -> A_Please:led rgb C7371893
- R22: value 1k2 -> 100
- SW1: value SW_Push -> ~; footprint Button_Switch_SMD:SW_SPST_SKQG_WithStem -> A_Please:switch C501547
- SW3: value SW_Push -> ~; footprint Button_Switch_SMD:SW_SPST_SKQG_WithStem -> A_Please:Sans titre
- moved SW2 130.1 mm to (82.0, 135.1), turned to -90 degrees
- moved SW1 126.8 mm to (93.0, 40.0), turned to 0 degrees
- moved D1 115.9 mm to (115.0, 40.0)
- moved R22 111.2 mm to (117.5, 60.9), turned to 90 degrees
- moved SW3 103.1 mm to (137.0, 43.0), turned to 0 degrees
- moved C46 84.1 mm to (139.2, 51.2), turned to 90 degrees
- moved J3 70.4 mm to (161.1, 104.2), turned to 0 degrees
- moved J1 68.1 mm to (161.1, 100.6), turned to 180 degrees
- moved C16 65.6 mm to (157.2, 100.6)
- moved R53 18.2 mm to (96.1, 70.6)
- moved R55 18.2 mm to (93.0, 70.6)
- moved R54 18.2 mm to (94.5, 70.6)
- moved J2 7.56 mm to (161.3, 44.1)
- moved C20 7.56 mm to (157.9, 45.1)
- moved R50 3.74 mm to (115.2, 70.6)
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- renumbered C3 to C10, C4 to C11, C5 to C12, C6 to C13, C7 to C14, C10 to C18, C11 to C20, C12 to C21, C15 to C24, C17 to C28, C18 to C29, C19 to C30, C20 to C31, C21 to C35, C22 to C36, C23 to C37, C24 to C38, C25 to C39, C26 to C40, C27 to C41, C28 to C42, C29 to C43, C30 to C44, C8 to C45, C31 to C47, C32 to C48, C33 to C49, C34 to C50, C35 to C51, C36 to C52, C37 to C53, C38 to C54, C39 to C55, C40 to C56, C41 to C57, C42 to C58, C1 to C8, C2 to C9, D10 to D4, D11 to D5, D12 to D6, D13 to D7, J4 to J3, J3 to J4, Q3 to Q1, Q7 to Q2, Q8 to Q3, Q9 to Q4, Q10 to Q5, R15 to R1, R62 to R10, R61 to R11, R63 to R12, R64 to R13, R66 to R14, R67 to R15, R69 to R16, R70 to R17, R72 to R18, R73 to R19, R65 to R2, R68 to R3, R6 to R30, R7 to R31, R8 to R32, R9 to R33, R10 to R34, R11 to R35, R12 to R36, R17 to R38, R18 to R39, R71 to R4, R24 to R40, R25 to R41, R26 to R42, R27 to R43, R28 to R44, R29 to R45, R30 to R46, R31 to R47, R32 to R48, R33 to R49, R74 to R5, R34 to R50, R35 to R51, R36 to R52, R37 to R53, R38 to R54, R39 to R55, R40 to R56, R41 to R57, R42 to R58, R43 to R59, R44 to R60, R45 to R61, R46 to R62, R47 to R63, R48 to R64, R49 to R65, R50 to R66, R51 to R67, R52 to R68, R53 to R69, R54 to R70, R55 to R71, R56 to R72, R57 to R73, R58 to R74, R59 to R75, R60 to R76, U8 to U7, U7 to U8
Connections:
- C16 pad 1: /RESET -> VBUS
- C46 pad 1: +3V3 -> PowerOnBP
- D1 pad 1: GND -> VBUS
- R22 pad 1: Net-(D8-A) -> /BLUE
- R22 pad 2: /LED FAIL -> Net-(Q8-G)
- SW1 pad 1: GND -> /BOOT
- SW1 pad 2: PowerOnBP -> +3V3
- SW2 pad 1: /BOOT -> GND
- SW2 pad 2: +3V3 -> DBG BP
- SW3 pad 1: GND -> unconnected-(SW3-Pad1)
- SW3 pad 2: DBG BP -> PowerOnBP
- U1 pad 2: /LED ON -> /RED
- U1 pad 3: /LED CONNECTÉ -> /GREEN
- U1 pad 4: /LED FAIL -> /BLUE
Routing:
- net +3V3: track 74.0 -> 541.6 mm, vias 0 -> 19
- net VBUS: track 251.1 -> 434.0 mm, vias 7 -> 10
- net /BOOT: track 2.23 -> 122.0 mm, vias 1 -> 6
- net PowerOnBP: track 1.86 -> 117.5 mm, vias 1 -> 4
- net /RESET: track 16.2 -> 126.8 mm, vias 1 -> 5
- net /RED: track 0.00 -> 90.5 mm, vias 0 -> 4
- net /GREEN: track 0.00 -> 89.6 mm, vias 0 -> 4
- net /BLUE: track 0.00 -> 88.3 mm, vias 0 -> 4
- net DBG LED: track 3.27 -> 69.6 mm, vias 1 -> 2
- net Vana: track 191.2 -> 243.6 mm, vias 10 -> 12
- net DBG BP: track 1.73 -> 18.9 mm, vias 1 -> 2
- net DBG IO1: track 2.67 -> 16.4 mm, vias 1 -> 2
- net Net-(Q8-D): track 0.00 -> 12.4 mm
- net DBG IO0: track 2.71 -> 14.6 mm, vias 1 -> 2
- net Net-(Q6-D): track 0.00 -> 11.6 mm
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- added copper zone on In2.Cu, net GND
Other:
- board text added: "REV A1.0"

Commit message: BIDIBOU
Parts:
- moved C18 3.35 mm to (93.8, 139.2), turned to 180 degrees
Routing:
- net DBG BP: track 18.9 -> 168.0 mm, vias 2 -> 11
- net DBG IO0: track 14.6 -> 133.5 mm, vias 2 -> 6
- net DBG RX: track 13.5 -> 130.0 mm, vias 2 -> 7
- net DBG TX: track 10.4 -> 120.5 mm, vias 2 -> 5
- net DBG IO1: track 16.4 -> 124.7 mm, vias 2 -> 1
- net /SWDIO: track 9.36 -> 79.3 mm, vias 1 -> 2
- net /SWCLK: track 12.7 -> 79.7 mm, vias 1 -> 2
- net DBG LED: track 69.6 -> 131.1 mm, vias 2 -> 3
- net /SDA: track 126.3 -> 186.6 mm, vias 3 -> 7
- net /SCL: track 128.0 -> 185.3 mm, vias 2 -> 6
- net /RESET: track 126.8 -> 180.1 mm, vias 5 -> 7
- net GND: track 10.3 -> 27.7 mm, vias 3 -> 117
- net VBUS: track 434.0 -> 451.4 mm, vias 10 -> 11
- net Vref USB: track 50.0 -> 52.7 mm
- net Vref ana: track 60.0 -> 62.3 mm
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