File: pcb/rev1/volume-mixer.kicad_sch (KiCad schematic)
At the start: 107 parts, among them CON1 TC2030-IDC, J1 Conn_01x10_Pin, J2 Conn_01x09_Pin, J3 Conn_01x09_Pin, J4 Conn_01x04_Pin, J5 Conn_01x04_Pin, J6 Conn_01x04_Pin, J7 Conn_01x04_Pin, J8 Conn_01x04_Pin, J9 Conn_01x04_Pin, Q1 2N7002, SW1 SW_Push, SW2 SW_Push, SW3 SW_Push, U1 STM32F302C8Tx, U2 24LC64, U3 XC6206PxxxMR, U4 XC6206PxxxMR, U5 PRTR5V0U2X, U6 TCA9548APWR, Y1 8MHz

Commit message: avancer du layout
Parts:
- removed C8, C9: 100nF, symbol Device:C_Small
- removed D2, D5, D6, D8: LED, symbol Device:LED
- removed J2, J3: Conn_01x09_Pin, symbol Connector:Conn_01x09_Pin
- removed Q1: 2N7002, Package_TO_SOT_SMD:SOT-23, symbol Transistor_FET:2N7002
- removed R16, R17, R19, R20, R22: 1k2, symbol Device:R_Small
- added D10, D11, D12, D13: LED, A_Please:LED C516299, symbol Device:LED
- added J3: Conn_01x10_Pin, Connector_PinHeader_1.27mm:PinHeader_2x05_P1.27mm_Vertical, symbol Connector:Conn_01x10_Pin
- added J4: Conn_01x04_Pin, Connector_PinHeader_2.54mm:PinHeader_1x04_P2.54mm_Vertical, symbol Connector:Conn_01x04_Pin
- added J5: JST, A_random_part:JST-SR-4, symbol Connector:Conn_01x04_Socket
- added Q1, Q10, Q3, Q7, Q8, Q9: NMOS, Package_TO_SOT_SMD:SOT-23, symbol Simulation_SPICE:NMOS
- added R15, R61, R64, R65, R67, R68, R70, R71, R73, R74: 100, Resistor_SMD:R_0603_1608Metric, symbol Device:R_Small
- added R62, R63, R66, R69, R72: 10K, Resistor_SMD:R_0603_1608Metric, symbol Device:R_Small
- C1, C2, C3, C4, C5, C6, C7: footprint Capacitor_SMD:C_0402_1005Metric -> Capacitor_SMD:C_0603_1608Metric
- C10: renamed from C12; footprint (none) -> Capacitor_SMD:C_0603_1608Metric
- C11: renamed from C13; footprint (none) -> Capacitor_SMD:C_0603_1608Metric
- C12: renamed from C14; footprint (none) -> Capacitor_SMD:C_0603_1608Metric
- C13: renamed from C15; value C_Small -> 100nF; footprint (none) -> Capacitor_SMD:C_0603_1608Metric
- C14: renamed from C16; footprint Capacitor_SMD:C_0402_1005Metric -> Capacitor_SMD:C_0603_1608Metric
- C15: renamed from C17; footprint (none) -> Capacitor_SMD:C_0603_1608Metric
- C16: renamed from C18; footprint Capacitor_SMD:C_0402_1005Metric -> Capacitor_SMD:C_0603_1608Metric
- C17: renamed from C19; footprint Capacitor_SMD:C_0402_1005Metric -> Capacitor_SMD:C_0603_1608Metric
- C18: renamed from C20; footprint Capacitor_SMD:C_0402_1005Metric -> Capacitor_SMD:C_0603_1608Metric
- C19: renamed from C21; footprint Capacitor_SMD:C_0402_1005Metric -> Capacitor_SMD:C_0603_1608Metric
- C20: renamed from C22; footprint Capacitor_SMD:C_0402_1005Metric -> Capacitor_SMD:C_0603_1608Metric
- C21: renamed from C23; footprint (none) -> Capacitor_SMD:C_0603_1608Metric
- C22: renamed from C24; footprint (none) -> Capacitor_SMD:C_0603_1608Metric
- C23: renamed from C25; footprint (none) -> Capacitor_SMD:C_0603_1608Metric
- C24: renamed from C26; footprint (none) -> Capacitor_SMD:C_0603_1608Metric
- C25: renamed from C27; footprint (none) -> Capacitor_SMD:C_0603_1608Metric
- C26: renamed from C28; footprint (none) -> Capacitor_SMD:C_0603_1608Metric
- C27: renamed from C29; footprint (none) -> Capacitor_SMD:C_0603_1608Metric
- C28: renamed from C30; footprint (none) -> Capacitor_SMD:C_0603_1608Metric
- C29: renamed from C31; footprint (none) -> Capacitor_SMD:C_0603_1608Metric
- C30: renamed from C32; footprint (none) -> Capacitor_SMD:C_0603_1608Metric
- C8: renamed from C11; footprint Capacitor_SMD:C_0402_1005Metric -> Capacitor_SMD:C_0603_1608Metric
- C9: renamed from C10; value C_Small -> 100nF; footprint (none) -> Capacitor_SMD:C_0603_1608Metric
- D1: renamed from D9; footprint (none) -> A_Please:LED C516299
- D3: footprint (none) -> A_Please:LED C516299
- J1: renamed from J4; footprint (none) -> Connector_PinHeader_2.54mm:PinHeader_1x04_P2.54mm_Vertical
- J10: renamed from J9; footprint (none) -> A_Please:Screen 0.91 I2C
- J2: renamed from J1; footprint (none) -> Connector_PinHeader_2.54mm:PinHeader_1x10_P2.54mm_Vertical
- J6: renamed from J5; footprint (none) -> A_Please:Screen 0.91 I2C
- J7: renamed from J6; footprint (none) -> A_Please:Screen 0.91 I2C
- J8: renamed from J7; footprint (none) -> A_Please:Screen 0.91 I2C
- J9: renamed from J8; footprint (none) -> A_Please:Screen 0.91 I2C
- R1, R2: value R_Small -> 10k; footprint (none) -> Resistor_SMD:R_0603_1608Metric
- R10, R24, R25, R26, R27, R28, R29, R30, R31, R32, R33, R34, R35, R36, R37, R38, R39, R6, R7, R8, R9: footprint (none) -> Resistor_SMD:R_0603_1608Metric
- R11, R12, R3, R4, R5: footprint Resistor_SMD:R_0402_1005Metric -> Resistor_SMD:R_0603_1608Metric
- R13: renamed from R23; footprint (none) -> Resistor_SMD:R_0603_1608Metric
- R16: renamed from R15; footprint (none) -> Resistor_SMD:R_0603_1608Metric
- R17: renamed from R13; footprint (none) -> Resistor_SMD:R_0603_1608Metric
- R18: renamed from R14; footprint (none) -> Resistor_SMD:R_0603_1608Metric
- R19: renamed from R18; footprint (none) -> Resistor_SMD:R_0603_1608Metric
- R22: renamed from R21; footprint (none) -> Resistor_SMD:R_0603_1608Metric
- SW1, SW3: footprint (none) -> Button_Switch_SMD:SW_SPST_SKQG_WithStem
- TP1, TP2, TP3, TP4, TP5: footprint (none) -> TestPoint:TestPoint_Keystone_5015_Micro_Mini
- U2: footprint (none) -> Package_SO:SOIC-8_3.9x4.9mm_P1.27mm
- renumbered D1 to D4, D4 to D5, D7 to D8
Connections:
- net +3V3: now also J3.1 (Pin_1), J4.1 (Pin_1)
- net D+: now also J5.3 (Pin_3)
- net D-: now also J5.2 (Pin_2)
- net GND: now also J3.3 (Pin_3), J3.5 (Pin_5), J3.9 (Pin_9), J4.4 (Pin_4), J5.4 (Pin_4), Q1.3 (S), Q10.3 (S), Q3.3 (S), Q7.3 (S), Q8.3 (S), Q9.3 (S), R62.1, R63.1, R66.1, R69.1, R72.1; no longer D3.1 (K)
- net Mute0Led: now also R61.1, R62.2
- net Mute1Led: now also R63.2, R64.1
- net Mute2Led: now also R66.2, R67.1
- net Mute3Led: now also R69.2, R70.1
- net Mute4Led: now also R72.2, R73.1
- net RESET: now also J3.10 (Pin_10), Q1.1 (D)
- net SCL: now also J4.2 (Pin_2)
- net SDA: now also J4.3 (Pin_3)
- net SWCLK: now also J3.4 (Pin_4)
- net SWDIO: now also J3.2 (Pin_2)
- net VBUS: now also J5.1 (Pin_1), R15.1, R65.1, R68.1, R71.1, R74.1
- net at C14.2, R5.1: now also Q1.2 (G)
- net at D3.2 (A): now also R15.2
- new net: D11.2 (A), R68.2
- new net: D13.1 (K), Q10.1 (D)
- new net: D13.2 (A), R74.2
- new net: D10.2 (A), R65.2
- new net: D11.1 (K), Q8.1 (D)
- new net: Q8.2 (G), R67.2
- new net: Q10.2 (G), R73.2
- new net: D10.1 (K), Q7.1 (D)
- new net: Q7.2 (G), R64.2
- new net: Q9.2 (G), R70.2
- new net: D12.1 (K), Q9.1 (D)
- new net: D12.2 (A), R71.2
- new net: D3.1 (K), Q3.1 (D)
- new net: Q3.2 (G), R61.2
- no-connect marks 2 -> 3
Other:
- note removed: "3V3 Decoupling"
- moved on the sheet: C1, C10, C12, C13, C14, C15, C16, C17, C18, C19, C2, C20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

Commit message: blabla
Connections:
- net SLIDER 0 mute : now also U1.40 (PB4); no longer U1.39 (PB3)
- net SLIDER 1 mute : now also U1.39 (PB3); no longer U1.40 (PB4)
- net SLIDER 3 mute : now also U1.26 (PB13); no longer U1.25 (PB12)
- net SLIDER 4 mute : now also U1.25 (PB12); no longer U1.26 (PB13)

Commit message: Capacitive sensor layout
Connections:
- net SliderSense1: now reaches R7.1, TP2.1
- net SliderSense4: now reaches R10.1, TP5.1
- net CapSense1: now reaches C15.1, U1.27 (PB14)
- net SliderSense2: now reaches R8.1, TP3.1
- net SliderSense0: now reaches R6.1, TP1.1
- net CapSense0: now reaches C10.1, U1.42 (PB6)
- net SliderSense3: now reaches R9.1, TP4.1
- net SLIDER 0 mute  renamed SLIDER_0_mute 
- net SLIDER 1 mute  renamed SLIDER_1_mute 
- net SLIDER 2 mute  renamed SLIDER_2_mute 
- net SLIDER 3 mute  renamed SLIDER_3_mute 
- net SLIDER 4 mute  renamed SLIDER_4_mute 
Other:
- moved on the sheet: C10, C15

Commit message: BIDIBOU
Connections:
- net Mute3Led: now also U1.20 (PB2); no longer U1.19 (PB1)
- net Mute4Led: now also U1.19 (PB1); no longer U1.20 (PB2)
Changed lines of the file:
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@@
 	(global_label "Mute3Led"
 		(shape input)
+		(at 67.31 81.28 180)
+		(fields_autoplaced yes)
+		(effects
+			(font
+				(size 1.27 1.27)
+			)
+			(justify right)
+		)
+		(property "Intersheetrefs" "${INTERSHEET_REFS}"
+			(at 55.4349 81.28 0)
+			(effects
+				(font
+					(size 1.27 1.27)
+				)
+				(justify right)
+				(hide yes)
+			)
+		)
+	)
+	(global_label "DBG RX"
+		(shape input)
+		(at 213.36 105.41 0)
+		(fields_autoplaced yes)
+		(effects
+			(font
+				(size 1.27 1.27)
+			)
+			(justify left)
+		)
+		(property "Intersheetrefs" "${INTERSHEET_REFS}"
+			(at 223.6023 105.41 0)
+			(effects
+				(font
+					(size 1.27 1.27)
+				)
+				(justify left)
+				(hide yes)
+			)
+		)
+	)
+	(global_label "Mute4Led"
+		(shape input)
 		(at 67.31 78.74 180)
 		(fields_autoplaced yes)
@@
 		)
 	)
-	(global_label "DBG RX"
-		(shape input)
-		(at 213.36 105.41 0)
-		(fields_autoplaced yes)
-		(effects
-			(font
-				(size 1.27 1.27)
-			)
-			(justify left)
-		)
-		(property "Intersheetrefs" "${INTERSHEET_REFS}"
-			(at 223.6023 105.41 0)
-			(effects
-				(font
-					(size 1.27 1.27)
-				)
-				(justify left)
+	(global_label "Mute2Led"
+		(shape input)
+		(at 67.31 114.3 180)
+		(fields_autoplaced yes)
+		(effects
+			(font
+				(size 1.27 1.27)
+			)
+			(justify right)
+		)
+		(property "Intersheetrefs" "${INTERSHEET_REFS}"
+			(at 55.4349 114.3 0)
+			(effects
+				(font
+					(size 1.27 1.27)
+				)
+				(justify right)
 				(hide yes)
 			)
@@
 	(global_label "Mute4Led"
 		(shape input)
-		(at 67.31 81.28 180)
-		(fields_autoplaced yes)
-		(effects
-			(font
-				(size 1.27 1.27)
-			)
-			(justify right)
-		)
-		(property "Intersheetrefs" "${INTERSHEET_REFS}"
-			(at 55.4349 81.28 0)
-			(effects
-				(font
-					(size 1.27 1.27)
-				)
-				(justify right)
-				(hide yes)
-			)
-		)
-	)
-	(global_label "Mute2Led"
-		(shape input)
-		(at 67.31 114.3 180)
-		(fields_autoplaced yes)
-		(effects
-			(font
-				(size 1.27 1.27)
-			)
-			(justify right)
-		)
-		(property "Intersheetrefs" "${INTERSHEET_REFS}"
-			(at 55.4349 114.3 0)
-			(effects
-				(font
-					(size 1.27 1.27)
-				)
-				(justify right)
-				(hide yes)
-			)
-		)
-	)
-	(global_label "Mute4Led"
-		(shape input)
 		(at 328.93 55.88 90)
 		(fields_autoplaced yes)
@@
 			)
 		)
-	)
-	(rule_area
-		(polyline
-			(pts
-				(xy 271.78 153.67) (xy 297.18 153.67) (xy 297.18 181.61) (xy 271.78 181.61)
-			)
-			(stroke
-				(width 0)
-				(type dash)
-			)
-			(fill
-				(type none)
-			)
-		)
-	)
-	(netclass_flag ""
-		(length 2.54)
-		(shape round)
-		(at 271.78 158.75 90)
-		(fields_autoplaced yes)
-		(effects
-			(font
-				(size 1.27 1.27)
-			)
-			(justify left bottom)
-		)
-		(property "Netclass" "Net_Isolé"
-			(at 269.24 158.0515 90)
-			(effects
-				(font
-					(size 1.27 1.27)
-				)
-				(justify left)
-			)
-		)
-		(property "Component Class" ""
-			(at -148.59 2.54 0)
-			(effects
-				(font
-					(size 1.27 1.27)
-					(italic yes)
-				)
-			)
-		)

Commit message: BIDIBOU
Parts:
- added C43, C44, C45, C46, C47, C48, C49, C50, C51, C52, C53, C54, C55, C56: 100nF, Capacitor_SMD:C_0603_1608Metric, symbol Device:C_Small
Connections:
- net +3V3: now also J1.3 (Pin_3), C43.1, C44.1, C45.1, C46.1; no longer J1.1 (Pin_1)
- net D+: now also U5.2 (IO1); no longer U5.3 (IO2)
- net D-: now also U5.3 (IO2); no longer U5.2 (IO1)
- net GND: now also C43.2, C44.2, C45.2, C46.2, C47.2, C48.2, C49.2, C50.2, C51.2, C52.2, C53.2, C54.2, C55.2, C56.2
- net VBUS: now also J1.1 (Pin_1), C48.1, C49.1, C50.1, C51.1, C52.1, C53.1, C54.1, C55.1, C56.1; no longer J1.3 (Pin_3)
- net Vana: now also C47.1
Other:
- moved on the sheet: CON1

Commit message: BIDIBOU
Parts:
- removed D4, D5, D8: LED, symbol Device:LED
- removed R16, R19: 1k2, Resistor_SMD:R_0603_1608Metric, symbol Device:R_Small
- removed SW1, SW2: SW_Push, Button_Switch_SMD:SW_SPST_SKQG_WithStem, symbol Switch:SW_Push
- added C1, C2: 100nF, Capacitor_SMD:C_0603_1608Metric, symbol Device:C_Small
- added D1: LED_ARGB, A_Please:led rgb C7371893, symbol Device:LED_ARGB
- added Q6, Q7, Q8: NMOS, Package_TO_SOT_SMD:SOT-23, symbol Simulation_SPICE:NMOS
- added R20, R21: 100, Resistor_SMD:R_0603_1608Metric, symbol Device:R_Small
- added R23, R24, R25: 10K, Resistor_SMD:R_0603_1608Metric, symbol Device:R_Small
- added R7: 150, Resistor_SMD:R_0603_1608Metric, symbol Device:R_Small
- added R8, R9: 95, Resistor_SMD:R_0603_1608Metric, symbol Device:R_Small
- added SW1: ~, A_Please:switch C501547, symbol Please:switch_GND
- added SW3: ~, A_Please:Sans titre, symbol Please:switch_led_C2848638
- D2: renamed from D1; footprint A_Please:LED C516299 -> LED_SMD:LED_0805_2012Metric
- R22: value 1k2 -> 100
- renumbered C3 to C10, C4 to C11, C5 to C12, C6 to C13, C7 to C14, C43 to C15, C48 to C16, C47 to C17, C10 to C18, C44 to C19, C11 to C20, C12 to C21, C13 to C22, C14 to C23, C15 to C24, C16 to C25, C46 to C26, C45 to C27, C17 to C28, C18 to C29, C51 to C3, C19 to C30, C20 to C31, C49 to C32, C50 to C33, C56 to C34, C21 to C35, C22 to C36, C23 to C37, C24 to C38, C25 to C39, C52 to C4, C26 to C40, C27 to C41, C28 to C42, C29 to C43, C30 to C44, C8 to C45, C9 to C46, C53 to C5, C54 to C6, C55 to C7, C1 to C8, C2 to C9, D10 to D4, D11 to D5, D12 to D6, D13 to D7, J4 to J3, J3 to J4, Q3 to Q1, Q7 to Q2, Q8 to Q3, Q9 to Q4, Q10 to Q5, Q1 to Q9, R15 to R1, R62 to R10, R61 to R11, R63 to R12, R64 to R13, R66 to R14, R67 to R15, R69 to R16, R70 to R17, R72 to R18, R73 to R19, R65 to R2, R2 to R26, R3 to R27, R4 to R28, R5 to R29, R68 to R3, R6 to R30, R7 to R31, R8 to R32, R9 to R33, R10 to R34, R11 to R35, R12 to R36, R1 to R37, R17 to R38, R18 to R39, R71 to R4, R24 to R40, R25 to R41, R26 to R42, R27 to R43, R28 to R44, R29 to R45, R30 to R46, R31 to R47, R32 to R48, R33 to R49, R74 to R5, R34 to R50, R35 to R51, R36 to R52, R37 to R53, R38 to R54, R39 to R55, R13 to R6, SW3 to SW2
Connections:
- net +3V3: now also SW1.2
- net BOOT: now also SW1.1
- net GND: now also C1.2, C2.2, Q6.3 (S), Q7.3 (S), Q8.3 (S), R23.1, R24.1, R25.1, SW1.3, SW3.4
- net PowerOnBP: now also SW3.2
- net VBUS: now also C1.1, C2.1, D1.1 (A)
- net BLUE: now reaches R22.1
- net BLUE: now also U1.4 (PC15), R25.2
- net LED CONNECTÉ renamed GREEN
- net GREEN: now also R21.1, R24.2
- net LED FAIL: no longer names the net of R22.2
- net LED FAIL: now also Q8.2 (G); no longer U1.4 (PC15)
- net LED ON renamed RED
- net RED: now also R20.1, R23.2
- new net: Q6.1 (D), R7.1
- new net: D1.2 (RK), R7.2
- new net: Q7.1 (D), R8.1
- new net: D1.3 (GK), R8.2
- new net: Q8.1 (D), R9.1
- new net: D1.4 (BK), R9.2
- new net: Q7.2 (G), R21.2
- new net: Q6.2 (G), R20.2
Other:
- moved on the sheet: C46, D2, R37, R6

Commit message: V1
Parts:
- C18, C24: footprint Capacitor_SMD:C_0603_1608Metric -> Capacitor_SMD:C_0805_2012Metric
- C8: value 4.7uF -> 4,7uF
Changed lines of the file:
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@@
 			)
 		)
-		(property "Footprint" "Capacitor_SMD:C_0603_1608Metric"
+		(property "Footprint" "Capacitor_SMD:C_0805_2012Metric"
 			(at 34.29 115.57 0)
 			(effects
@@
 			)
 		)
-		(property "Value" "4.7uF"
+		(property "Value" "4,7uF"
 			(at 25.4 35.5662 0)
 			(effects
@@
 			)
 		)
-		(property "Footprint" "Capacitor_SMD:C_0603_1608Metric"
+		(property "Footprint" "Capacitor_SMD:C_0805_2012Metric"
 			(at 34.29 95.25 0)
 			(effects

Commit message: imagine ça marche
Parts:
- added H1, H2: MountingHole_Pad, A_Please:Vis M2.5, symbol Mechanical:MountingHole_Pad
Connections:
- net GND: now also H1.1, H2.1
